File: hw/sch_pcb/SOLARMINI01B.kicad_pcb (KiCad board)
At the start: 2 copper layers, 40.1 x 40.1 mm, 28 parts, among them J1 WAGO 256, J2 WAGO 256, J3 HEADER_1x01, J4 HEADER_2x03_PARALLEL, M1 HOLE, M2 HOLE, M3 HOLE, M4 HOLE, U1 SPV1040

Commit message: Úpravy PCB a generování výrobních dat.
Other:
- rule pad_to_mask_clearance: 0 -> 0.15

Commit message: Edit BOM
Parts:
- J1: value WAGO 256 -> WAGO 256 RED
- J2: value WAGO 256 -> WAGO 256 BLUE
Changed lines of the file:
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@@
     (property "Sheetfile" "SOLARMINI01B.kicad_sch")
     (property "Sheetname" "")
+    (property "UST_ID" "5c70984412875079b91f87c3")
     (attr through_hole)
     (fp_text reference "J2" (at -5.842 0 90) (layer "F.SilkS")
       (effects (font (size 1.524 1.524) (thickness 0.3048)))
     )
-    (fp_text value "WAGO 256" (at 0.254 4.064) (layer "F.SilkS") hide
+    (fp_text value "WAGO 256 BLUE" (at 0.254 4.064) (layer "F.SilkS") hide
       (effects (font (size 1.524 1.524) (thickness 0.3048)))
     )
@@
     (property "Sheetfile" "SOLARMINI01B.kicad_sch")
     (property "Sheetname" "")
+    (property "UST_ID" "5c70984412875079b91f87c5")
     (attr through_hole)
     (fp_text reference "J1" (at -5.842 0 90) (layer "F.SilkS")
       (effects (font (size 1.524 1.524) (thickness 0.3048)))
     )
-    (fp_text value "WAGO 256" (at 0.254 4.064) (layer "F.SilkS") hide
+    (fp_text value "WAGO 256 RED" (at 0.254 4.064) (layer "F.SilkS") hide
       (effects (font (size 1.524 1.524) (thickness 0.3048)))
     )
@@
     (property "Sheetfile" "SOLARMINI01B.kicad_sch")
     (property "Sheetname" "")
+    (property "UST_ID" "5c70984412875079b91f8867")
     (attr smd)
     (fp_text reference "C7" (at 0 2.85) (layer "B.SilkS")
@@
     (property "Sheetfile" "SOLARMINI01B.kicad_sch")
     (property "Sheetname" "")
+    (property "UST_ID" "5c70984512875079b91f898c")
     (attr smd)
     (fp_text reference "R1" (at 0 1.65 90) (layer "B.SilkS") hide
@@
     (property "Sheetfile" "SOLARMINI01B.kicad_sch")
     (property "Sheetname" "")
+    (property "UST_ID" "5c70984712875079b91f8b45")
     (attr smd)
     (fp_text reference "C8" (at 0 1.68 90) (layer "B.SilkS") hide
@@
     (property "Sheetfile" "SOLARMINI01B.kicad_sch")
     (property "Sheetname" "")
+    (property "UST_ID" "5c70984712875079b91f8b50")
     (attr smd)
     (fp_text reference "C3" (at -2.8092 0.4064) (layer "B.SilkS")
@@
     (property "Sheetfile" "SOLARMINI01B.kicad_sch")
     (property "Sheetname" "")
+    (property "UST_ID" "5c70984712875079b91f8aa0")
     (attr smd)
     (fp_text reference "R8" (at 0 1.65 90) (layer "B.SilkS") hide
@@
     (property "Sheetfile" "SOLARMINI01B.kicad_sch")
     (property "Sheetname" "")
+    (property "UST_ID" "5c70984412875079b91f8867")
     (attr smd)
     (fp_text reference "C1" (at 0 2.85 90) (layer "B.SilkS") hide
@@
     (property "Sheetfile" "SOLARMINI01B.kicad_sch")
     (property "Sheetname" "")
+    (property "UST_ID" "5c70984712875079b91f8aa6")
     (attr smd)
     (fp_text reference "R7" (at 0 1.65) (layer "B.SilkS")
@@
     (property "Sheetfile" "SOLARMINI01B.kicad_sch")
     (property "Sheetname" "")
+    (property "UST_ID" "5c70984712875079b91f8b4c")
     (attr smd)
     (fp_text reference "C4" (at 0 1.68 90) (layer "B.SilkS") hide
@@
     (property "Sheetfile" "SOLARMINI01B.kicad_sch")
     (property "Sheetname" "")
+    (property "UST_ID" "5c70984812875079b91f8bbd")
     (attr smd)
     (fp_text reference "C5" (at 0 1.68 90) (layer "B.SilkS") hide
@@
     (property "Sheetfile" "SOLARMINI01B.kicad_sch")
     (property "Sheetname" "")
+    (property "UST_ID" "5c70984512875079b91f88c7")
     (attr smd)
     (fp_text reference "D2" (at -3.556 0.0254) (layer "B.SilkS") hide
@@
     (property "Sheetfile" "SOLARMINI01B.kicad_sch")
     (property "Sheetname" "")
+    (property "UST_ID" "60be2ed51287500165e6c1cd")
     (attr smd)
     (fp_text reference "R6" (at 0 1.82 90) (layer "B.SilkS") hide
@@
     (property "Sheetfile" "SOLARMINI01B.kicad_sch")
     (property "Sheetname" "")
+    (property "UST_ID" "5c70984512875079b91f88b0")
     (attr smd)
     (fp_text reference "D1" (at 0 2.5) (layer "B.SilkS")
@@
     (property "Sheetfile" "SOLARMINI01B.kicad_sch")
     (property "Sheetname" "")
+    (property "UST_ID" "5c70984612875079b91f89bc")
     (attr smd)
     (fp_text reference "U1" (at 0 2.45 90) (layer "B.SilkS") hide
@@
     (property "Sheetfile" "SOLARMINI01B.kicad_sch")
     (property "Sheetname" "")
+    (property "UST_ID" "5c70984512875079b91f898c")
     (attr smd)
     (fp_text reference "R5" (at -0.0508 -1.9558 90) (layer "B.SilkS")
@@
     (property "Sheetfile" "SOLARMINI01B.kicad_sch")
     (property "Sheetname" "")
+    (property "UST_ID" "5c70984512875079b91f896b")
     (attr smd)
     (fp_text reference "R3" (at 0 1.65 90) (layer "B.SilkS")
@@
     (property "Sheetfile" "SOLARMINI01B.kicad_sch")
     (property "Sheetname" "")
+    (property "UST_ID" "5c70984512875079b91f898c")
     (attr smd)
     (fp_text reference "R4" (at 0 1.65 90) (layer "B.SilkS")
@@
     (property "Sheetfile" "SOLARMINI01B.kicad_sch")
     (property "Sheetname" "")
+    (property "UST_ID" "5c70984712875079b91f8b4c")
     (attr smd)
     (fp_text reference "C2" (at 0 1.68 90) (layer "B.SilkS") hide
@@
     (property "Sheetfile" "SOLARMINI01B.kicad_sch")
     (property "Sheetname" "")
+    (property "UST_ID" "5c70984412875079b91f8867")
     (attr smd)
     (fp_text reference "C6" (at -8.636 2.247 90) (layer "B.SilkS") hide
@@
     (property "Sheetfile" "SOLARMINI01B.kicad_sch")
     (property "Sheetname" "")
+    (property "UST_ID" "5c70984412875079b91f8822")
     (attr through_hole)
     (fp_text reference "L1" (at 0 0) (layer "B.SilkS")
