File: hw/sch_pcb/SOLARMINI01B.kicad_sch (KiCad schematic)
At the start: 27 parts, among them J1 WAGO 256, J2 WAGO 256, J3 HEADER_1x01, J4 HEADER_2x03_PARALLEL, M1 HOLE, M2 HOLE, M3 HOLE, M4 HOLE, U1 SPV1040

Commit message: edit schema
Parts:
- added C?: 1nF, symbol Device:C
- C2: value 1nF -> 100nF
Connections:
- net GND: now also C?.2
- net at R7.1, R8.2, U1.5 (VCTRL): now also C?.1
Changed lines of the file:
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@@
   (junction (at 126.365 92.075) (diameter 0) (color 0 0 0 0))
   (junction (at 126.365 103.505) (diameter 0) (color 0 0 0 0))
+  (junction (at 126.365 107.315) (diameter 0) (color 0 0 0 0))
   (junction (at 137.16 69.85) (diameter 0) (color 0 0 0 0))
   (junction (at 150.495 69.85) (diameter 0) (color 0 0 0 0))
@@
     (stroke (width 0) (type default) (color 0 0 0 0))
   )
-  (wire (pts (xy 120.65 107.315) (xy 207.645 107.315))
+  (wire (pts (xy 120.65 107.315) (xy 126.365 107.315))
     (stroke (width 0) (type default) (color 0 0 0 0))
   )
@@
   )
   (wire (pts (xy 126.365 103.505) (xy 126.365 101.6))
+    (stroke (width 0) (type default) (color 0 0 0 0))
+  )
+  (wire (pts (xy 126.365 107.315) (xy 207.645 107.315))
+    (stroke (width 0) (type default) (color 0 0 0 0))
+  )
+  (wire (pts (xy 126.365 109.22) (xy 126.365 107.315))
+    (stroke (width 0) (type default) (color 0 0 0 0))
+  )
+  (wire (pts (xy 126.365 119.38) (xy 126.365 116.84))
     (stroke (width 0) (type default) (color 0 0 0 0))
   )
@@
     (pin "1")
   )
+  (symbol (lib_id "power:GND") (at 126.365 119.38 0) (unit 1)
+    (in_bom yes) (on_board yes) (fields_autoplaced)
+    (property "Reference" "#PWR?" (id 0) (at 126.365 125.73 0)
+      (effects (font (size 1.27 1.27)) hide)
+    )
+    (property "Value" "GND" (id 1) (at 126.365 123.9424 0))
+    (property "Footprint" "" (id 2) (at 126.365 119.38 0)
+      (effects (font (size 1.27 1.27)) hide)
+    )
+    (property "Datasheet" "" (id 3) (at 126.365 119.38 0)
+      (effects (font (size 1.27 1.27)) hide)
+    )
+    (pin "1")
+  )
   (symbol (lib_id "power:GND") (at 137.16 80.01 0) (unit 1)
     (in_bom yes) (on_board yes) (fields_autoplaced)
@@
       (effects (font (size 1.27 1.27)) (justify left))
     )
-    (property "Value" "1nF" (id 1) (at 81.026 114.8966 0)
+    (property "Value" "100nF" (id 1) (at 81.026 114.8966 0)
       (effects (font (size 1.27 1.27)) (justify left))
     )
@@
     )
     (property "Datasheet" "~" (id 3) (at 126.365 97.79 0)
+      (effects (font (size 1.27 1.27)) hide)
+    )
+    (pin "1")
+    (pin "2")
+  )
+  (symbol (lib_id "Device:C") (at 126.365 113.03 0) (unit 1)
+    (in_bom yes) (on_board yes) (fields_autoplaced)
+    (property "Reference" "C?" (id 0) (at 129.286 112.1215 0)
+      (effects (font (size 1.27 1.27)) (justify left))
+    )
+    (property "Value" "1nF" (id 1) (at 129.286 114.8966 0)
+      (effects (font (size 1.27 1.27)) (justify left))
+    )
+    (property "Footprint" "" (id 2) (at 127.3302 116.84 0)
+      (effects (font (size 1.27 1.27)) hide)
+    )
+    (property "Datasheet" "~" (id 3) (at 126.365 113.03 0)
       (effects (font (size 1.27 1.27)) hide)
     )
@@
       (reference "#PWR012") (unit 1) (value "GND") (footprint "")
     )
+    (path "/243ed74a-f275-427a-a73c-017b1ab626fc"
+      (reference "#PWR?") (unit 1) (value "GND") (footprint "")
+    )
     (path "/88af01fd-14b2-4407-87ca-8afa17bc9491"
       (reference "C1") (unit 1) (value "47uF/16") (footprint "")
     )
     (path "/a6860e4f-d3f8-4bc9-97d6-895c5ce84032"
-      (reference "C2") (unit 1) (value "1nF") (footprint "")
+      (reference "C2") (unit 1) (value "100nF") (footprint "")
     )
     (path "/c752bd8f-f7fd-4c60-891e-9b87bb99e626"
@@
       (reference "C7") (unit 1) (value "47uF/16") (footprint "")
     )
+    (path "/f95fbc88-beda-47e0-825b-8cd3c63256d1"
+      (reference "C?") (unit 1) (value "1nF") (footprint "")
+    )
     (path "/6ebf9b32-12cd-4595-af06-e4cf81ac4d0a"

Commit message: Edit PCB
Parts:
- C1, C6, C7: footprint (none) -> Mlab_C:TantalC_SizeC_Reflow
- C2, C3, C4, C5: footprint (none) -> Capacitor_SMD:C_0805_2012Metric
- C8: renamed from C?; footprint (none) -> Capacitor_SMD:C_0805_2012Metric
- D1, D2: footprint (none) -> Diode_SMD:D_SMA
- J3: footprint (none) -> Mlab_Pin_Headers:Straight_1x01
- J4: footprint (none) -> Mlab_Pin_Headers:Straight_2x03
- L1: footprint (none) -> Mlab_L:DE1205-10
- M1, M2, M3, M4: footprint Mlab_Mechanical:dira_3mm -> Mlab_Mechanical:MountingHole_3mm
- R1, R2, R3, R4, R5, R7, R8: footprint (none) -> Resistor_SMD:R_0805_2012Metric
- R6: footprint (none) -> Resistor_SMD:R_1206_3216Metric
Connections:
- no-connect marks 0 -> 4

Commit message: Edit BOM
Parts:
- C1, C6, C7: UST_ID (none) -> 5c70984412875079b91f8867
- C2, C4: UST_ID (none) -> 5c70984712875079b91f8b4c
- C3: UST_ID (none) -> 5c70984712875079b91f8b50
- C5: UST_ID (none) -> 5c70984812875079b91f8bbd
- C8: UST_ID (none) -> 5c70984712875079b91f8b45
- D1: UST_ID (none) -> 5c70984512875079b91f88b0
- D2: UST_ID (none) -> 5c70984512875079b91f88c7
- J1: value WAGO 256 -> WAGO 256 RED; UST_ID (none) -> 5c70984412875079b91f87c5
- J2: value WAGO 256 -> WAGO 256 BLUE; UST_ID (none) -> 5c70984412875079b91f87c3
- L1: UST_ID (none) -> 5c70984412875079b91f8822
- R1, R4, R5: UST_ID (none) -> 5c70984512875079b91f898c
- R3: UST_ID (none) -> 5c70984512875079b91f896b
- R6: UST_ID (none) -> 60be2ed51287500165e6c1cd
- R7: UST_ID (none) -> 5c70984712875079b91f8aa6
- R8: UST_ID (none) -> 5c70984712875079b91f8aa0
- U1: UST_ID (none) -> 5c70984612875079b91f89bc
Changed lines of the file:
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@@
+      (effects (font (size 1.27 1.27)) hide)
+    )
+    (property "UST_ID" "5c70984412875079b91f8822" (id 4) (at 87.63 88.265 0)
       (effects (font (size 1.27 1.27)) hide)
     )
@@
     (in_bom yes) (on_board yes)
     (property "Reference" "J1" (id 0) (at 42.545 86.4384 0))
-    (property "Value" "WAGO 256" (id 1) (at 35.56 85.725 0)
+    (property "Value" "WAGO 256 RED" (id 1) (at 35.56 85.725 0)
       (effects (font (size 1.016 1.016)) hide)
     )
@@
     (property "Datasheet" "" (id 3) (at 36.83 85.725 0)
       (effects (font (size 1.524 1.524)))
+    )
+    (property "UST_ID" "5c70984412875079b91f87c5" (id 4) (at 38.1 86.995 0)
+      (effects (font (size 1.27 1.27)) hide)
     )
     (pin "1")
@@
     (in_bom yes) (on_board yes)
     (property "Reference" "J2" (id 0) (at 42.545 108.0284 0))
-    (property "Value" "WAGO 256" (id 1) (at 35.56 107.315 0)
+    (property "Value" "WAGO 256 BLUE" (id 1) (at 35.56 107.315 0)
       (effects (font (size 1.016 1.016)) hide)
     )
@@
       (effects (font (size 1.524 1.524)))
     )
+    (property "UST_ID" "5c70984412875079b91f87c3" (id 4) (at 38.1 108.585 0)
+      (effects (font (size 1.27 1.27)) hide)
+    )
     (pin "1")
   )
@@
       (effects (font (size 1.27 1.27)) hide)
     )
+    (property "UST_ID" "5c70984512875079b91f898c" (id 4) (at 67.31 100.965 0)
+      (effects (font (size 1.27 1.27)) hide)
+    )
     (pin "1")
     (pin "2")
@@
     )
     (property "Datasheet" "~" (id 3) (at 91.44 100.33 0)
+      (effects (font (size 1.27 1.27)) hide)
+    )
+    (property "UST_ID" "5c70984512875079b91f896b" (id 4) (at 91.44 100.33 0)
       (effects (font (size 1.27 1.27)) hide)
     )
@@
       (effects (font (size 1.27 1.27)) hide)
     )
+    (property "UST_ID" "5c70984512875079b91f898c" (id 4) (at 137.16 92.075 0)
+      (effects (font (size 1.27 1.27)) hide)
+    )
     (pin "1")
     (pin "2")
@@
       (effects (font (size 1.27 1.27)) hide)
     )
+    (property "UST_ID" "5c70984512875079b91f898c" (id 4) (at 137.16 103.505 0)
+      (effects (font (size 1.27 1.27)) hide)
+    )
     (pin "1")
     (pin "2")
@@
       (effects (font (size 1.27 1.27)) hide)
     )
+    (property "UST_ID" "60be2ed51287500165e6c1cd" (id 4) (at 196.85 69.85 0)
+      (effects (font (size 1.27 1.27)) hide)
+    )
     (pin "1")
     (pin "2")
@@
       (effects (font (size 1.27 1.27)) hide)
     )
+    (property "UST_ID" "5c70984712875079b91f8aa6" (id 4) (at 207.645 99.695 0)
+      (effects (font (size 1.27 1.27)) hide)
+    )
     (pin "1")
     (pin "2")
@@
     )
     (property "Datasheet" "~" (id 3) (at 207.645 111.76 0)
+      (effects (font (size 1.27 1.27)) hide)
+    )
+    (property "UST_ID" "5c70984712875079b91f8aa0" (id 4) (at 207.645 111.76 0)
       (effects (font (size 1.27 1.27)) hide)
     )
@@
       (effects (font (size 1.27 1.27)) hide)
     )
+    (property "UST_ID" "5c70984512875079b91f88b0" (id 4) (at 107.315 77.47 0)
+      (effects (font (size 1.27 1.27)) hide)
+    )
     (pin "1")
     (pin "2")
@@
       (effects (font (size 1.27 1.27)) hide)
     )
+    (property "UST_ID" "5c70984512875079b91f88c7" (id 4) (at 161.925 75.565 0)
+      (effects (font (size 1.27 1.27)) hide)
+    )
     (pin "1")
     (pin "2")
@@
       (effects (font (size 1.27 1.27)) hide)
     )
+    (property "UST_ID" "5c70984412875079b91f8867" (id 4) (at 52.705 102.235 0)
+      (effects (font (size 1.27 1.27)) hide)
+    )
     (pin "1")
     (pin "2")
@@
       (effects (font (size 1.27 1.27)) hide)
     )
+    (property "UST_ID" "5c70984712875079b91f8b4c" (id 4) (at 78.105 113.03 0)
+      (effects (font (size 1.27 1.27)) hide)
+    )
     (pin "1")
     (pin "2")
@@
       (effects (font (size 1.27 1.27)) hide)
     )
+    (property "UST_ID" "5c70984712875079b91f8b50" (id 4) (at 126.365 97.79 0)
+      (effects (font (size 1.27 1.27)) hide)
+    )
     (pin "1")
     (pin "2")
@@
       (effects (font (size 1.27 1.27)) hide)
     )
+    (property "UST_ID" "5c70984712875079b91f8b45" (id 4) (at 126.365 113.03 0)
+      (effects (font (size 1.27 1.27)) hide)
+    )
     (pin "1")
     (pin "2")
@@
       (effects (font (size 1.27 1.27)) hide)
     )
+    (property "UST_ID" "5c70984712875079b91f8b4c" (id 4) (at 137.16 74.93 0)
+      (effects (font (size 1.27 1.27)) hide)
+    )
     (pin "1")
     (pin "2")
@@
       (effects (font (size 1.27 1.27)) hide)
     )
+    (property "UST_ID" "5c70984812875079b91f8bbd" (id 4) (at 150.495 74.93 0)
+      (effects (font (size 1.27 1.27)) hide)
+    )
     (pin "1")
     (pin "2")
@@
       (effects (font (size 1.27 1.27)) hide)
     )
+    (property "UST_ID" "5c70984412875079b91f8867" (id 4) (at 175.895 75.565 0)
+      (effects (font (size 1.27 1.27)) hide)
+    )
     (pin "1")
     (pin "2")
@@
     )
     (property "Datasheet" "~" (id 3) (at 214.63 75.565 0)
+      (effects (font (size 1.27 1.27)) hide)
+    )
+    (property "UST_ID" "5c70984412875079b91f8867" (id 4) (at 214.63 75.565 0)
       (effects (font (size 1.27 1.27)) hide)
     )
@@
     )
     (property "Datasheet" "" (id 3) (at 107.95 94.615 0)
+      (effects (font (size 1.27 1.27)) hide)
+    )
+    (property "UST_ID" "5c70984612875079b91f89bc" (id 4) (at 107.95 94.615 0)
       (effects (font (size 1.27 1.27)) hide)
     )
@@
     )
     (path "/ae7443a5-830b-41de-a85d-f96b896b066d"
-      (reference "J1") (unit 1) (value "WAGO 256") (footprint "Mlab_CON:WAGO256")
+      (reference "J1") (unit 1) (value "WAGO 256 RED") (footprint "Mlab_CON:WAGO256")
     )
     (path "/f4b72ede-6abb-4b6e-a92b-9fe98fd3ac59"
-      (reference "J2") (unit 1) (value "WAGO 256") (footprint "Mlab_CON:WAGO256")
+      (reference "J2") (unit 1) (value "WAGO 256 BLUE") (footprint "Mlab_CON:WAGO256")
     )
     (path "/f9262074-7be4-480f-9dc1-dcf7e5e55044"

Commit message: Update module documentation.
Other:
- note added: "## Photovoltaic pannel connection Usually array of four cells in series with following parameters: Isc = 2,3 A Voc= 2,5 V Impp= 2,1 A Vmpp= 2,1 V Pm= 4,4 Wp"
- title: (none) -> SOLARMINI01B
